File: src/schematics/multi-channel-preamp/multi-channel-preamp.kicad_sch (KiCad schematic)
At the start: 21 parts, among them J1 Channel 1 Input, J10 Channel 2 Output, J11 Power 6.6V Heater, J2 Ch 1 Volume, J3 Ch 1 Bypass Cap, J4 Channel 1 Output, J5 B+, J6 Channel 2 Input, J8 Ch 2 Bypass Cap, J9 Ch 2 Volume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

Commit message: git cleanup
Parts:
- J11: value Power 6.6V Heater -> Power 6.3V Heater
- U1: footprint Valve:Valve_ECC-83-1 -> OL Library:BELTON_VT9-PT Fat Pad
Changed lines of the file:
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@@
 			)
 		)
-		(property "Value" "Power 6.6V Heater"
+		(property "Value" "Power 6.3V Heater"
 			(at 223.52 20.9549 90)
 			(effects
@@
 			)
 		)
-		(property "Footprint" "Valve:Valve_ECC-83-1"
+		(property "Footprint" "OL Library:BELTON_VT9-PT Fat Pad"
 			(at 214.122 38.1 0)
 			(effects
@@
 			)
 		)
-		(property "Footprint" "Valve:Valve_ECC-83-1"
+		(property "Footprint" "OL Library:BELTON_VT9-PT Fat Pad"
 			(at 128.778 63.5 0)
 			(effects
@@
 			)
 		)
-		(property "Footprint" "Valve:Valve_ECC-83-1"
+		(property "Footprint" "OL Library:BELTON_VT9-PT Fat Pad"
 			(at 126.238 137.16 0)
 			(effects
