File: src/schematics/multi-channel-preamp/multi-channel-preamp.kicad_pcb (KiCad board)
At the start: 2 copper layers, 95.3 x 102.9 mm, 21 parts, among them J1 Channel 1 Input, J10 Channel 2 Output, J11 Power 6.6V Heater, J2 Ch 1 Volume, J3 Ch 1 Bypass Cap, J4 Channel 1 Output, J5 B+, J6 Channel 2 Input, J8 Ch 2 Bypass Cap, J9 Ch 2 Volume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

Commit message: git cleanup
Parts:
- J1: value Channel 1 Input -> Ch 1 Input
- J10: value Channel 2 Output -> Ch 2 Output
- J4: value Channel 1 Output -> Ch 1 Output
- J6: value Channel 2 Input -> Ch 2 Input
- U1: footprint Valve:Valve_ECC-83-1 -> OL Library:BELTON_VT9-PT Fat Pad
- moved R3 20.0 mm to (91.4, 71.1)
- moved R5 18.8 mm to (146.1, 101.6)
- moved J6 15.3 mm to (138.4, 113.0)
- moved R7 15.3 mm to (151.1, 104.1)
- moved J8 12.1 mm to (149.9, 92.3)
- moved R2 10.2 mm to (97.8, 72.4)
- moved J1 10.2 mm to (105.4, 62.2)
- moved R8 9.40 mm to (132.1, 116.5)
- moved R4 8.52 mm to (113.0, 58.4)
- moved U1 8.37 mm to (123.2, 87.3), turned to -90 degrees
- moved J3 7.69 mm to (94.9, 82.6)
- moved J4 7.62 mm to (149.9, 77.5)
- moved J10 7.25 mm to (94.9, 96.3)
- moved R6 4.22 mm to (140.5, 95.2)
- moved C2 2.88 mm to (125.5, 126.7)
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Routing:
- net Net-(U1A-A): track 56.0 -> 37.7 mm
- net Net-(U1B-A): track 47.1 -> 36.1 mm
- net Net-(J3-Pin_2): track 34.8 -> 44.2 mm
- net Net-(J8-Pin_2): track 34.8 -> 44.1 mm
- net Net-(J11-Pin_2): track 36.1 -> 42.6 mm
- net Net-(J2-Pin_2): track 11.5 -> 17.6 mm
- net Net-(J11-Pin_1): track 20.7 -> 15.6 mm
- net Net-(U1B-G): track 12.8 -> 7.72 mm
- net Net-(J6-Pin_1): track 25.5 -> 20.7 mm
- net Net-(J10-Pin_2): track 12.5 -> 17.2 mm
- net Net-(U1A-G): track 12.9 -> 8.47 mm
- net Net-(J1-Pin_1): track 22.0 -> 19.9 mm
- net Net-(J5-Pin_2): track 87.5 -> 85.9 mm
Other:
- board size 95.3 x 102.9 mm -> 74.9 x 90.2 mm

Commit message: big add
Parts:
- J1: value Ch 1 Input -> Channel 1 Input
- J10: value Ch 2 Output -> Channel 2 Output
- J11: value Power 6.6V Heater -> Heater
- J4: value Ch 1 Output -> Channel 1 Output
- J6: value Ch 2 Input -> Channel 2 Input
- moved C2 15.5 mm to (125.5, 111.1)
- moved C1 14.0 mm to (118.1, 62.2)
- moved J2 13.3 mm to (143.9, 49.1)
- moved J5 13.3 mm to (125.7, 48.9)
- moved J11 12.4 mm to (119.6, 125.1)
- moved J9 12.4 mm to (99.2, 125.1)
Routing:
- net Net-(U1A-A): track 37.7 -> 21.7 mm
- net Net-(U1B-A): track 36.1 -> 20.5 mm
- net Net-(J11-Pin_2): track 42.6 -> 56.6 mm
- net Net-(J11-Pin_1): track 15.6 -> 28.0 mm
- net Net-(J5-Pin_2): track 85.9 -> 97.9 mm
- net Net-(J2-Pin_2): track 17.6 -> 28.6 mm
- net Net-(J10-Pin_2): track 17.2 -> 27.7 mm
Other:
- outline, holes or cut-outs redrawn
- board text added: "4S Universal Preamp 2024-06-26"
