File: src/schematics/tapeop-output/tapeop-output.kicad_pcb (KiCad board)
At the start: 2 copper layers, 80 x 63.5 mm, 11 parts, among them J1 Heater Supply, J2 B+, J3 VOUT, J4 VIN, U1 ECC83

Commit message: big add
Other:
- outline, holes or cut-outs redrawn
Changed lines of the file:
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@@
 		(property ki_fp_filters "TerminalBlock*:*")
 		(sheetname "Root")
-		(sheetfile "multi-channel-preamp-output.kicad_sch")
+		(sheetfile "tapeop-output.kicad_sch")
 		(attr through_hole)
 		(fp_line
@@
 		(property ki_fp_filters "TerminalBlock*:*")
 		(sheetname "Root")
-		(sheetfile "multi-channel-preamp-output.kicad_sch")
+		(sheetfile "tapeop-output.kicad_sch")
 		(attr through_hole)
 		(fp_line
@@
 		(property ki_fp_filters "R_*")
 		(sheetname "Root")
-		(sheetfile "multi-channel-preamp-output.kicad_sch")
+		(sheetfile "tapeop-output.kicad_sch")
 		(attr through_hole)
 		(fp_line
@@
 		(property ki_fp_filters "VALVE*NOVAL*P*")
 		(sheetname "Root")
-		(sheetfile "multi-channel-preamp-output.kicad_sch")
+		(sheetfile "tapeop-output.kicad_sch")
 		(attr through_hole)
 		(fp_line
@@
 		(fp_arc
 			(start -7.8 8.31)
-			(mid -8.564506 7.522323)
+			(mid -8.564507 7.522324)
 			(end -9.25 6.665)
 			(stroke
@@
 		(fp_arc
 			(start -9.25 -6.665)
-			(mid -8.564507 -7.522323)
+			(mid -8.564506 -7.522323)
 			(end -7.8 -8.31)
 			(stroke
@@
 		(fp_arc
 			(start 2.6 -11.0967)
-			(mid 3.655918 -10.796814)
+			(mid 3.655918 -10.796815)
 			(end 4.67823 -10.3971)
 			(stroke
@@
 		(property ki_fp_filters "TerminalBlock*:*")
 		(sheetname "Root")
-		(sheetfile "multi-channel-preamp-output.kicad_sch")
+		(sheetfile "tapeop-output.kicad_sch")
 		(attr through_hole)
 		(fp_line
@@
 		(property ki_fp_filters "TerminalBlock*:*")
 		(sheetname "Root")
-		(sheetfile "multi-channel-preamp-output.kicad_sch")
+		(sheetfile "tapeop-output.kicad_sch")
 		(attr through_hole)
 		(fp_line
@@
 		(property ki_fp_filters "R_*")
 		(sheetname "Root")
-		(sheetfile "multi-channel-preamp-output.kicad_sch")
+		(sheetfile "tapeop-output.kicad_sch")
 		(attr through_hole)
 		(fp_line
@@
 		(property ki_fp_filters "C_*")
 		(sheetname "Root")
-		(sheetfile "multi-channel-preamp-output.kicad_sch")
+		(sheetfile "tapeop-output.kicad_sch")
 		(attr through_hole)
 		(fp_line
@@
 		(property ki_fp_filters "R_*")
 		(sheetname "Root")
-		(sheetfile "multi-channel-preamp-output.kicad_sch")
+		(sheetfile "tapeop-output.kicad_sch")
 		(attr through_hole)
 		(fp_line
@@
 		(property ki_fp_filters "R_*")
 		(sheetname "Root")
-		(sheetfile "multi-channel-preamp-output.kicad_sch")
+		(sheetfile "tapeop-output.kicad_sch")
 		(attr through_hole)
 		(fp_line
@@
 		(property ki_fp_filters "C_*")
 		(sheetname "Root")
-		(sheetfile "multi-channel-preamp-output.kicad_sch")
+		(sheetfile "tapeop-output.kicad_sch")
 		(attr through_hole)
 		(fp_line
@@
 	(gr_circle
 		(center 93.98 109.22)
-		(end 96.52 110.49)
+		(end 95.48 109.22)
 		(stroke
 			(width 0.05)
@@
 	(gr_circle
 		(center 93.98 55.88)
-		(end 96.52 57.15)
+		(end 95.48 55.88)
 		(stroke
 			(width 0.05)
@@
 	(gr_circle
 		(center 163.83 55.88)
-		(end 166.37 57.15)
+		(end 165.33 55.88)
 		(stroke
 			(width 0.05)
@@
 	(gr_circle
 		(center 163.83 109.22)
-		(end 166.37 110.49)
+		(end 165.33 109.22)
 		(stroke
 			(width 0.05)
@@
 		)
 	)
+	(dimension
+		(type aligned)
+		(layer "F.Cu")
+		(pts
+			(xy 90.17 52.07) (xy 90.17 113.03)
+		)
+		(height -2.54)
+		(gr_text "60.9600 mm"
+			(at 90.91 82.55 90)
+			(layer "F.Cu")
+			(effects
+				(font
+					(size 1.5 1.5)
+					(thickness 0.3)
+				)
+			)
+		)
+		(format
+			(prefix "")
+			(suffix "")
+			(units 3)
+			(units_format 1)
+			(precision 4)
+		)
+		(style
+			(thickness 0.2)
+			(arrow_length 1.27)
+			(text_position_mode 0)
+			(extension_height 0.58642)
+			(extension_offset 0.5) keep_text_aligned)
+	)
+	(dimension
+		(type aligned)
+		(layer "F.Cu")
+		(pts
+			(xy 142.24 107.95) (xy 154.94 107.95)
+		)
+		(height 3.81)
+		(gr_text "12.7000 mm"
+			(at 148.59 110.49 0)
+			(layer "F.Cu")
+			(effects
+				(font
+					(size 1.5 1.5)
+					(thickness 0.3)
+				)
+			)
+		)
+		(format
+			(prefix "")
+			(suffix "")
+			(units 3)
+			(units_format 1)
+			(precision 4)
+		)
+		(style
+			(thickness 0.2)
+			(arrow_length 1.27)
+			(text_position_mode 2)
+			(extension_height 0.58642)
+			(extension_offset 0.5) keep_text_aligned)
+	)
 	(segment
