File: src/schematics/pultec-three-band-eq/pultec-three-band-eq.kicad_pcb (KiCad board)
At the start: 2 copper layers, 159.5 x 120 mm, 85 parts, among them J1 IN, J10 Lo Boost Sel Ret, J11 Lo Boost Lvl, J12 Hi Cut Sel Ret, J13 Hi Boost Sel Snd, J14 Mid bst/cut switch, J15 Mid Sel Ret, J16 Mid Sel Ret, J17 2H, J18 1H, J19 Hi Boost Sel Ret, J2 OUT, J20 Hi Boost Q, J21 Hi Boost Lvl, J22 100mH, J23 200mH, J24 300mH, J25 600mH, J26 .45H, J27 .22H, J28 .1H, J29 Mid Lvl (47 Log), J3 Hi Cut Sel Snd, J30 Mid Sel Snd, J4 Hi Cut Lvl, J5 Lo Cut Sel Snd, J6 Lo Boost Sel Snd, J7 Low Cut Lvl, J8 Hi Boost Sel Rtn, J9 Low Cut Sel Ret

Commit message: - re-worked the mid-range - exported gerbers for PCB manufacture
Parts:
- removed C42: 1n5, OL Library:C_Rect_L7.0mm_W2.0mm_P5.00mm_Fat_Pad
- removed C43, C45: 4n7, OL Library:C_Rect_L7.0mm_W2.0mm_P5.00mm_Fat_Pad
- removed C44, C46: 2n2, OL Library:C_Rect_L7.0mm_W2.0mm_P5.00mm_Fat_Pad
- removed J16: Mid Sel Ret, OL Library:TerminalBlock_Phoenix_MKDS-1,5-12_1x12_P5.00mm_Horizontal_Fat_Pad
- removed J17: 2H, OL Library:TerminalBlock_Phoenix_MKDS-1,5-2_1x02_P5.00mm_Horizontal Fat Pad
- removed J18: 1H, OL Library:TerminalBlock_Phoenix_MKDS-1,5-2_1x02_P5.00mm_Horizontal Fat Pad
- removed J22: 100mH, OL Library:TerminalBlock_Phoenix_MKDS-1,5-2_1x02_P5.00mm_Horizontal Fat Pad
- removed J23: 200mH, OL Library:TerminalBlock_Phoenix_MKDS-1,5-2_1x02_P5.00mm_Horizontal Fat Pad
- removed J24: 300mH, OL Library:TerminalBlock_Phoenix_MKDS-1,5-2_1x02_P5.00mm_Horizontal Fat Pad
- removed J25: 600mH, OL Library:TerminalBlock_Phoenix_MKDS-1,5-2_1x02_P5.00mm_Horizontal Fat Pad
- removed J26: .45H, OL Library:TerminalBlock_Phoenix_MKDS-1,5-2_1x02_P5.00mm_Horizontal Fat Pad
- removed J27: .22H, OL Library:TerminalBlock_Phoenix_MKDS-1,5-2_1x02_P5.00mm_Horizontal Fat Pad
- removed J28: .1H, OL Library:TerminalBlock_Phoenix_MKDS-1,5-2_1x02_P5.00mm_Horizontal Fat Pad
- removed J30: Mid Sel Snd, OL Library:TerminalBlock_Phoenix_MKDS-1,5-2_1x02_P5.00mm_Horizontal Fat Pad
- removed R4: 100K, OL Library:R_Axial_DIN0207_L6.3mm_D2.5mm_P7.62mm_Horizontal
- removed R5: 4K7, OL Library:R_Axial_DIN0207_L6.3mm_D2.5mm_P7.62mm_Horizontal
- removed R6: 1K, OL Library:R_Axial_DIN0207_L6.3mm_D2.5mm_P7.62mm_Horizontal
- added J31: Mid In, OL Library:TerminalBlock_Phoenix_MKDS-1,5-2_1x02_P5.00mm_Horizontal Fat Pad, F.Cu at (53.2, 33.2)
- added J32: Mid Out, OL Library:TerminalBlock_Phoenix_MKDS-1,5-2_1x02_P5.00mm_Horizontal Fat Pad, F.Cu at (192.0, 114.6)
- added J35: Mid L Sel Ret/C Sel Snd, OL Library:TerminalBlock_Phoenix_MKDS-1,5-2_1x02_P5.00mm_Horizontal Fat Pad, F.Cu at (196.0, 128.7)
- added J36: Mid C Sel Ret, OL Library:TerminalBlock_Phoenix_MKDS-1,5-6_1x06_P5.00mm_Horizontal_Fat_Pad, F.Cu at (146.8, 81.3)
- added J38: Mid Cut/Bst Sw, OL Library:TerminalBlock_Phoenix_MKDS-1,5-3_1x03_P5.00mm_Horizontal Fat Pad, F.Cu at (192.0, 103.5)
- added J39: Mid Cut Q, OL Library:TerminalBlock_Phoenix_MKDS-1,5-3_1x03_P5.00mm_Horizontal Fat Pad, F.Cu at (192.0, 87.3)
- added J40: Mid L Ret, OL Library:TerminalBlock_Phoenix_MKDS-1,5-12_1x12_P5.00mm_Horizontal_Fat_Pad, F.Cu at (137.3, 45.6)
- C10: value 47n -> Mid C2A
- C11: value 22n -> Mid C2B
- C12: value 22n -> Mid C3A
- C13: value 12n -> Mid C3B
- C36: value 12n -> Mid C4A
- C37: value 2n2 -> Mid C4B
- C38: value 3n3 -> Mid C5A
- C39: value 3n3 -> Mid C5B
- C40: value 1n -> Mid C6A
- C41: value 4n7 -> Mid C6B
- C8: value 33n -> Mid C1A
- C9: value 150n -> Mid C1B
- J14: value Mid bst/cut switch -> Mid L Sel send; footprint OL Library:TerminalBlock_Phoenix_MKDS-1,5-3_1x03_P5.00mm_Horizontal Fat Pad -> OL Library:TerminalBlock_Phoenix_MKDS-1,5-12_1x12_P5.00mm_Horizontal_Fat_Pad
- J15: value Mid Sel Ret -> Hi Boost L Snd; footprint OL Library:TerminalBlock_Phoenix_MKDS-1,5-2_1x02_P5.00mm_Horizontal Fat Pad -> TerminalBlock_Phoenix:TerminalBlock_Phoenix_MKDS-1,5-6_1x06_P5.00mm_Horizontal
- moved J14 112.2 mm to (137.4, 34.0), turned to 0 degrees
- moved J15 66.2 mm to (129.5, 101.7)
- moved C38 31.4 mm to (179.6, 61.2), turned to 0 degrees
- moved C39 26.5 mm to (179.6, 67.2), turned to 0 degrees
- moved C13 19.5 mm to (159.9, 66.9), turned to 0 degrees
- moved C9 17.9 mm to (139.7, 66.6), turned to 0 degrees
- moved C10 13.5 mm to (149.8, 60.8), turned to 0 degrees
- moved C8 13.1 mm to (139.7, 60.6), turned to 0 degrees
- moved C41 11.8 mm to (189.2, 66.9), turned to 0 degrees
- moved C11 11.7 mm to (149.8, 66.8), turned to 0 degrees
- moved C37 9.06 mm to (169.8, 66.9), turned to 0 degrees
- moved C40 6.18 mm to (189.2, 60.9), turned to 0 degrees
- moved C12 5.85 mm to (159.9, 60.9), turned to 0 degrees
- moved C36 4.75 mm to (169.8, 60.9), turned to 0 degrees
Connections:
- C10 pad 1: Net-(J17-Pin_1) -> Net-(J36-Pin_2)
- C10 pad 2: Net-(J16-Pin_3) -> Net-(J38-Pin_2)
- C11 pad 1: Net-(J17-Pin_1) -> Net-(J36-Pin_2)
- C11 pad 2: Net-(J16-Pin_4) -> Net-(J38-Pin_2)
- C12 pad 1: Net-(J18-Pin_1) -> Net-(J36-Pin_3)
- C12 pad 2: Net-(J16-Pin_5) -> Net-(J38-Pin_2)
- C13 pad 1: Net-(J18-Pin_1) -> Net-(J36-Pin_3)
- C13 pad 2: Net-(J16-Pin_6) -> Net-(J38-Pin_2)
- C14 pad 1: Net-(J25-Pin_1) -> Net-(J15-Pin_4)
- C15 pad 1: Net-(J24-Pin_1) -> Net-(J15-Pin_3)
- C16 pad 1: Net-(J24-Pin_1) -> Net-(J15-Pin_3)
- C17 pad 1: Net-(J23-Pin_1) -> Net-(J15-Pin_2)
- C2a2 pad 1: Net-(J24-Pin_1) -> Net-(J15-Pin_3)
- C34 pad 1: Net-(J22-Pin_1) -> Net-(J15-Pin_1)
- C35 pad 1: Net-(J22-Pin_1) -> Net-(J15-Pin_1)
- C36 pad 1: Net-(J26-Pin_1) -> Net-(J36-Pin_4)
- C36 pad 2: Net-(J16-Pin_7) -> Net-(J38-Pin_2)
- C37 pad 1: Net-(J26-Pin_1) -> Net-(J36-Pin_4)
- C37 pad 2: Net-(J16-Pin_7) -> Net-(J38-Pin_2)
- C38 pad 1: Net-(J17-Pin_1) -> Net-(J36-Pin_5)
- C38 pad 2: Net-(J16-Pin_4) -> Net-(J38-Pin_2)
- C39 pad 1: Net-(J18-Pin_1) -> Net-(J36-Pin_5)
- C39 pad 2: Net-(J16-Pin_5) -> Net-(J38-Pin_2)
- C40 pad 1: Net-(J28-Pin_1) -> Net-(J36-Pin_6)
- C40 pad 2: Net-(J16-Pin_11) -> Net-(J38-Pin_2)
- C41 pad 1: Net-(J26-Pin_1) -> Net-(J36-Pin_6)
- C41 pad 2: Net-(J16-Pin_8) -> Net-(J38-Pin_2)
- C4a2 pad 1: Net-(J23-Pin_1) -> Net-(J15-Pin_2)
- C5a2 pad 1: Net-(J22-Pin_1) -> Net-(J15-Pin_1)
- C8 pad 1: Net-(J17-Pin_1) -> Net-(J36-Pin_1)
- C8 pad 2: Net-(J16-Pin_1) -> Net-(J38-Pin_2)
- C9 pad 1: Net-(J17-Pin_1) -> Net-(J36-Pin_1)
- C9 pad 2: Net-(J16-Pin_2) -> Net-(J38-Pin_2)
- J15 pad 1: Net-(J14-Pin_2) -> Net-(J15-Pin_1)
- J15 pad 2: Net-(J14-Pin_2) -> Net-(J15-Pin_2)
- J29 pad 1: Net-(J29-Pin_1) -> /pultec-mid-band/MID OUT
- J29 pad 2: Net-(J29-Pin_1) -> /pultec-mid-band/MID L SND
- J29 pad 3: /HI BOOST OUT -> /OUT
Routing:
- net /pultec-mid-band/MID OUT: track 0.00 -> 177.7 mm, vias 0 -> 1
- net Net-(J38-Pin_2): track 0.00 -> 145.8 mm
- net Net-(J17-Pin_1): track 126.4 -> 0.00 mm
- net Net-(J18-Pin_1): track 97.9 -> 0.00 mm
- net Net-(J26-Pin_1): track 71.9 -> 0.00 mm
- net Net-(J27-Pin_1): track 67.2 -> 0.00 mm
- net Net-(J16-Pin_8): track 44.7 -> 0.00 mm
- net Net-(J16-Pin_11): track 41.4 -> 0.00 mm
- net Net-(J22-Pin_1): track 37.7 -> 0.00 mm
- net /OUT: track 57.7 -> 94.7 mm
- net Net-(J16-Pin_5): track 36.6 -> 0.00 mm
- net Net-(J24-Pin_1): track 34.0 -> 0.00 mm
- net Net-(J15-Pin_1): track 0.00 -> 33.4 mm
- net Net-(J15-Pin_3): track 0.00 -> 32.7 mm
- net Net-(J15-Pin_4): track 0.00 -> 32.5 mm
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Other:
- board text added: "HB Lvl"
- board text added: "HB Q"
- board text added: "HB Sel Ret"
- board text added: "HB Sel Snd"
- board text added: "HC Sel Ret"
- board text added: "HC Sel Snd"
- board text added: "Hi Boost L Send"
- board text added: "Hi Boost Sel Return"
- board text added: "Hi Cut Lvl"
- board text added: "IN"
- board text added: "LB Sel Snd"
- board text added: "Lo Boost Sel Ret"
- board text added: "Lo Boost Sel Snd"
- board text added: "Lo Bst Lvl"
- board text added: "Lo Cut Lvl"
- board text added: "M Cut Q"
- board text added: "M Cut/Bst"
- board text added: "M L Sel Ret"
- board text added: "Mid IN"
- board text added: "Mid L Ret"
- board text added: "Mid L Sel Snd"
- board text added: "Mid Lvl (47 Log)"
- board text added: "Mid OUT"
- board text added: "OUT"
